File: magnetic/hardware/magnetometer/magnetometer.kicad_sch (KiCad schematic)
At the start: 18 parts, among them J1 Conn_01x04_Socket, J2 Conn_01x04_Socket, U1 MLX90393SLW-ABA-011-RE, U2 MLX90393SLW-ABA-011-RE, U3 MLX90393SLW-ABA-011-RE, U4 MLX90393SLW-ABA-011-RE

Commit message: annotation fixes
Parts:
- removed C9: 0.1uF, Capacitor_SMD:C_0402_1005Metric_Pad0.74x0.62mm_HandSolder, symbol Device:C
- added C7: 0.1uF, Capacitor_SMD:C_0402_1005Metric_Pad0.74x0.62mm_HandSolder, symbol Device:C
- renumbered C7 to C2, C8 to C3, C2 to C4, C3 to C5, C4 to C6, C5 to C8, D2 to D1
Connections:
- net +3.3V: now also C7.1
- net GND: now also C7.2
